Commit message: Agrega parámetros faltantes del modelo
Se ordenan los archivos del modelo

File: vtol_description/urdf/ciii_vtol.xacro (robot description, xacro)
@@ -1,7 +1,14 @@
 <?xml version="1.0"?>
 <robot name="ciii1dvtol" xmlns:xacro="http://www.ros.org/wiki/xacro">
+    <!-- Import RViz colors -->
     <xacro:include filename="$(find vtol_description)/urdf/material.xacro" />
+    <!-- Gazebo elements (colors) -->
+    <xacro:include filename="$(find vtol_description)/urdf/ciii_vtol.gazebo" />
+    <!-- Robot parameters file -->
+    <xacro:include filename="$(find vtol_description)/urdf/params.xacro" />
+    <!-- Macro for VTOL lateral parts -->
     <xacro:include filename="$(find vtol_description)/urdf/lateral.xacro" />
-    <xacro:include filename="$(find vtol_description)/urdf/params.xacro" />
+    <!-- Fixed world link -->
+    <link name="world_link" />
     <!-- Base -->
     <link name="base_link">
@@ -26,4 +33,8 @@
         </inertial>
     </link>
+    <joint name="world_link" type="fixed">
+        <parent link="world_link" />
+        <child link="base_link" />
+    </joint>
     <!-- Laterals -->
     <xacro:vtol_lateral name="front" origin_xyz="0 -0.019 0.150" />

File: vtol_description/urdf/material.xacro (robot description, xacro)
@@ -5,16 +5,3 @@
         <color rgba="0.6 0.5 0.2 1" />
     </material>
-    <!-- Gazebo materials -->
-    <gazebo reference="base_link">
-        <material>Gazebo/Wood</material>
-    </gazebo>
-    <gazebo reference="front_link">
-        <material>Gazebo/Wood</material>
-    </gazebo>
-    <gazebo reference="rear_link">
-        <material>Gazebo/Wood</material>
-    </gazebo>
-    <gazebo reference="crossbar_link">
-        <material>Gazebo/Wood</material>
-    </gazebo>
 </robot>

File: vtol_description/urdf/params.xacro (robot description, xacro)
@@ -23,3 +23,12 @@
     <xacro:property name="L_Iyy" value="${(1/12) * L_mass * (L_x**2 + L_z**2)}" />
     <xacro:property name="L_Izz" value="${(1/12) * L_mass * (L_x**2 + L_y**2)}" />
+    <!-- Crossbar -->
+    <xacro:property name="C_x" value="0.050" />
+    <xacro:property name="C_y" value="0.047" />
+    <xacro:property name="C_z" value="0.009" />
+    <xacro:property name="C_vol" value="${C_x * C_y * C_z}" />
+    <xacro:property name="C_mass" value="${1000.0 * C_vol * rho_mdf}" />
+    <xacro:property name="C_Ixx" value="${(1/12) * C_mass * (C_y**2 + C_z**2)}" />
+    <xacro:property name="C_Iyy" value="${(1/12) * C_mass * (C_x**2 + C_z**2)}" />
+    <xacro:property name="C_Izz" value="${(1/12) * C_mass * (C_x**2 + C_y**2)}" />
 </robot>

Commit message: Agrega soporte del eje al modelo del robot

File: vtol_description/urdf/ciii_vtol.xacro (robot description, xacro)
@@ -67,3 +67,35 @@
         <child link="crossbar_link" />
     </joint>
+    <!-- Axis suppport (front & rear) -->
+    <link name="support_link">
+        <visual>
+            <origin xyz="0 0 0" rpy="0 0 0" />
+            <geometry>
+                <mesh filename="package://vtol_description/meshes/axis_support.stl" />
+            </geometry>
+            <material name="blue" />
+        </visual>
+        <collision>
+            <origin xyz="0 0 0.013" rpy="0 0 0" />
+            <geometry>
+                <box size="0.050 0.026 0.042" />
+            </geometry>
+        </collision>
+        <inertial>
+            <origin xyz="0 0 0.016" rpy="0 0 0" />
+            <mass value="0.068250" />
+            <inertia ixx="0.000013878" ixy="0" ixz="0"
+                iyy="0.000024252" iyz="0" izz="0.000018064" />
+        </inertial>
+        -->
+    </link>
+    <joint name="support_joint" type="continuous">
+        <!--
+        <dynamics damping="0.001" friction="0.001" />
+        -->
+        <origin xyz="0 0 0.150" rpy="0 0 0" />
+        <parent link="base_link" />
+        <child link="support_link" />
+        <axis xyz="0 1 0" />
+    </joint>
 </robot>

File: vtol_description/urdf/material.xacro (robot description, xacro)
@@ -3,5 +3,8 @@
     <!-- RViz materials -->
     <material name="brown" >
-        <color rgba="0.6 0.5 0.2 1" />
+        <color rgba="${150/255} ${130/255} ${50/255} 1" />
+    </material>
+    <material name="blue">
+        <color rgba="0 0 ${200/255} 1" />
     </material>
 </robot>

Commit message: Agrega barra principal al modelo del robot

File: vtol_description/urdf/ciii_vtol.xacro (robot description, xacro)
@@ -99,3 +99,28 @@
         <axis xyz="0 1 0" />
     </joint>
+    <!-- Main bar -->
+    <link name="bar_link">
+        <visual xyz="0 0 0" rpy="0 0 0">
+            <origin xyz="0 0 0.016" rpy="0 0 0" />
+            <geometry>
+                <box size="${MB_L} ${MB_w_out} ${MB_w_out}" rpy="0 0 0"/>
+            </geometry>
+            <material name="white" />
+        </visual>
+        <collision>
+            <origin xyz="0 0 0.016" rpy="0 0 0" />
+            <geometry>
+                <box size="${MB_L} ${MB_w_out} ${MB_w_out}" rpy="0 0 0"/>
+            </geometry>
+        </collision>
+        <inertial>
+            <origin xyz="0 0 0" rpy="0 0 0" />
+            <mass value="${MB_mass}" />
+            <inertia ixx="${MB_Ixx}" ixy="0" ixz="0" iyy="${MB_Iyy}" iyz="0" izz="${MB_Iyy}" />
+        </inertial>
+    </link>
+    <joint name="bar_joint" type="fixed">
+        <parent link="support_link" />
+        <child link="bar_link" />
+    </joint>
 </robot>

File: vtol_description/urdf/material.xacro (robot description, xacro)
@@ -8,3 +8,6 @@
         <color rgba="0 0 ${200/255} 1" />
     </material>
+    <material name="white" >
+        <color rgba="1 1 1 1" />
+    </material>
 </robot>

File: vtol_description/urdf/params.xacro (robot description, xacro)
@@ -32,3 +32,13 @@
     <xacro:property name="C_Iyy" value="${(1/12) * C_mass * (C_x**2 + C_z**2)}" />
     <xacro:property name="C_Izz" value="${(1/12) * C_mass * (C_x**2 + C_y**2)}" />
+    <!-- Main bar -->
+    <xacro:property name="MB_rho" value="2.7" />
+    <xacro:property name="MB_w_out" value="0.020" />
+    <xacro:property name="MB_thickness" value="0.0016" />
+    <xacro:property name="MB_w_in" value="${MB_w_out - 2*MB_thickness}" />
+    <xacro:property name="MB_L" value="0.500" />
+    <xacro:property name="MB_vol" value="${(MB_w_out**2 - MB_w_in**2) * MB_L}" />
+    <xacro:property name="MB_mass" value="${1000.0 * MB_vol * MB_rho}" />
+    <xacro:property name="MB_Ixx" value="${(1/12) * MB_mass * 2 * MB_w_out**2}" />
+    <xacro:property name="MB_Iyy" value="${(1/12) * MB_mass * (MB_w_out**2 + MB_L**2)}" />
 </robot>

Commit message: Agrega motores al modelo del robot

File: vtol_description/urdf/ciii_vtol.xacro (robot description, xacro)
@@ -9,4 +9,6 @@
     <!-- Macro for VTOL lateral parts -->
     <xacro:include filename="$(find vtol_description)/urdf/lateral.xacro" />
+    <!-- Macro for brushless motors -->
+    <xacro:include filename="$(find vtol_description)/urdf/motor.xacro" />
     <!-- Fixed world link -->
     <link name="world_link" />
@@ -124,3 +126,6 @@
         <child link="bar_link" />
     </joint>
+    <!-- Left & Right motor -->
+    <xacro:motor name="lmotor" origin_xyz="-0.225 0 0.0435" />
+    <xacro:motor name="rmotor" origin_xyz="0.225 0 0.0435" />
 </robot>

File: vtol_description/urdf/material.xacro (robot description, xacro)
@@ -11,3 +11,6 @@
         <color rgba="1 1 1 1" />
     </material>
+    <material name="gray">
+        <color rgba="${80/255} ${80/255} ${80/255} 1" />
+    </material>
 </robot>

Commit message: Agrega hélices al modelo del robot

File: vtol_description/urdf/ciii_vtol.xacro (robot description, xacro)
@@ -7,8 +7,8 @@
     <!-- Robot parameters file -->
     <xacro:include filename="$(find vtol_description)/urdf/params.xacro" />
-    <!-- Macro for VTOL lateral parts -->
+    <!-- Macro for VTOL parts (lateral, motor and propeller -->
     <xacro:include filename="$(find vtol_description)/urdf/lateral.xacro" />
-    <!-- Macro for brushless motors -->
     <xacro:include filename="$(find vtol_description)/urdf/motor.xacro" />
+    <xacro:include filename="$(find vtol_description)/urdf/propeller.xacro" />
     <!-- Fixed world link -->
     <link name="world_link" />
@@ -126,6 +126,9 @@
         <child link="bar_link" />
     </joint>
-    <!-- Left & Right motor -->
+    <!-- Left & Right motors -->
     <xacro:motor name="lmotor" origin_xyz="-0.225 0 0.0435" />
     <xacro:motor name="rmotor" origin_xyz="0.225 0 0.0435" />
+    <!-- Left & Right propellers -->
+    <xacro:propeller name="lprop" parent="lmotor" />
+    <xacro:propeller name="rprop" parent="rmotor" />
 </robot>

File: vtol_description/urdf/material.xacro (robot description, xacro)
@@ -14,3 +14,6 @@
         <color rgba="${80/255} ${80/255} ${80/255} 1" />
     </material>
+    <material name="yellow">
+        <color rgba="${255/255} ${220/255} ${0/255} 1" />
+    </material>
 </robot>

Commit message: Modifica modelo del robot para usar 'ros_control'

File: vtol_description/urdf/ciii_vtol.xacro (robot description, xacro)
@@ -1,4 +1,4 @@
 <?xml version="1.0"?>
-<robot name="ciii1dvtol" xmlns:xacro="http://www.ros.org/wiki/xacro">
+<robot name="ciiivtol" xmlns:xacro="http://www.ros.org/wiki/xacro">
     <!-- Import RViz colors -->
     <xacro:include filename="$(find vtol_description)/urdf/material.xacro" />
@@ -95,4 +95,5 @@
         <!--
         <dynamics damping="0.001" friction="0.001" />
+        <limit effort="30.0" velocity="10.0" lower="${-20.0 * pi / 180.0}" upper="${20.0 * pi / 180.0}" />
         -->
         <origin xyz="0 0 0.150" rpy="0 0 0" />

File: vtol_description/urdf/motor.xacro (robot description, xacro)
@@ -29,5 +29,5 @@
             </inertial>
         </link>
-        <joint name="${name}_join" type="fixed">
+        <joint name="${name}_joint" type="fixed">
             <origin xyz="${origin_xyz}" rpy="0 0 0" />
             <parent link="bar_link" />

File: vtol_description/urdf/propeller.xacro (robot description, xacro)
@@ -27,5 +27,5 @@
             </inertial>
         </link>
-        <joint name="${name}_join" type="continuous">
+        <joint name="${name}_joint" type="continuous">
             <origin xyz="0 0 0" rpy="0 0 0" />
             <parent link="${parent}_link" />

Commit message: Agrega IMU

File: vtol_description/urdf/ciii_vtol.xacro (robot description, xacro)
@@ -3,6 +3,4 @@
     <!-- Import RViz colors -->
     <xacro:include filename="$(find vtol_description)/urdf/material.xacro" />
-    <!-- Gazebo elements (colors) -->
-    <xacro:include filename="$(find vtol_description)/urdf/ciii_vtol.gazebo" />
     <!-- Robot parameters file -->
     <xacro:include filename="$(find vtol_description)/urdf/params.xacro" />
@@ -11,4 +9,6 @@
     <xacro:include filename="$(find vtol_description)/urdf/motor.xacro" />
     <xacro:include filename="$(find vtol_description)/urdf/propeller.xacro" />
+    <!-- Gazebo elements materials and plugins -->
+    <xacro:include filename="$(find vtol_description)/urdf/ciii_vtol.gazebo" />
     <!-- Fixed world link -->
     <link name="world_link" />
@@ -133,3 +133,29 @@
     <xacro:propeller name="lprop" parent="lmotor" />
     <xacro:propeller name="rprop" parent="rmotor" />
+    <!-- IMU sensor -->
+    <link name="imu_link">
+        <visual xyz="0 0 0" rpy="0 0 0">
+            <origin xyz="0 0 0" rpy="0 0 0" />
+            <geometry>
+                <box size="0.02 0.02 0.01" />
+            </geometry>
+            <material name="gray" />
+        </visual>
+        <collision>
+            <origin xyz="0 0 0" rpy="0 0 0" />
+            <geometry>
+                <box size="0.02 0.02 0.01" />
+            </geometry>
+        </collision>
+        <inertial>
+            <origin xyz="0 0 0" rpy="0 0 0" />
+            <mass value="0.001" />
+            <inertia ixx="0.000001" ixy="0" ixz="0" iyy="0.000001" iyz="0" izz="0.000001"/>
+        </inertial>
+    </link>
+    <joint name="imu_joint" type="fixed">
+        <origin xyz="0 0 0.05" />
+        <parent link="bar_link" />
+        <child link="imu_link" />
+    </joint>
 </robot>
